File: KiCad/FA-Merus-Amplifier/FA-Merus-Amplifier.kicad_pcb (KiCad board)
At the start: 2 copper layers, 80 x 43 mm, 63 parts, among them J100 Conn_02x10_Odd_Even, J101 Conn_01x02_Male, J102 Conn_01x02_Male, J103 Conn_01x02_Male, U200 MA120x0P

Commit message: Update for release
Parts:
- added Q100: BC846BW, Package_TO_SOT_SMD:SOT-323_SC-70, F.Cu at (-27.8, 6.50)
- added R100: 10k, Resistor_SMD:R_0402_1005Metric, F.Cu at (-30.5, 6.00)
- added R216: 0R, Resistor_SMD:R_0402_1005Metric, F.Cu at (-13.8, 0.50)
- added R217: 0R, Resistor_SMD:R_0402_1005Metric, F.Cu at (-13.8, -0.50)
- added R218: 0R, Resistor_SMD:R_0402_1005Metric, F.Cu at (-13.8, -2.50)
- added R219: 0R, Resistor_SMD:R_0402_1005Metric, F.Cu at (-13.8, -1.50)
- added R220: 0R, Resistor_SMD:R_0402_1005Metric, F.Cu at (-13.8, -4.50)
- added R221: 0R, Resistor_SMD:R_0402_1005Metric, F.Cu at (-13.8, -3.50)
- added R222: 2.2k, Resistor_SMD:R_0402_1005Metric, F.Cu at (-13.8, 3.50)
- added R223: 2.2k, Resistor_SMD:R_0402_1005Metric, F.Cu at (-13.8, 2.50)
- FB201, FB202, FB203, FB204: value 600R -> BLE32PN300SN1L; footprint Inductor_SMD:L_1206_3216Metric -> Inductor_SMD:L_1210_3225Metric
- FB205: value 600R -> BLE32PN300SN1L; footprint Inductor_SMD:L_1806_4516Metric -> Inductor_SMD:L_1210_3225Metric
- J101: value Conn_01x02_Male -> JST_XH_S2B-XH-A; footprint Connector_JST:JST_PH_S2B-PH-SM4-TB_1x02-1MP_P2.00mm_Horizontal -> Connector_JST:JST_XH_S2B-XH-A_1x02_P2.50mm_Horizontal
- J102, J103: value Conn_01x02_Male -> JST_XH_S3B-XH-A; footprint Connector_JST:JST_PH_S2B-PH-SM4-TB_1x02-1MP_P2.00mm_Horizontal -> Connector_JST:JST_XH_S3B-XH-A_1x03_P2.50mm_Horizontal
- PCB100: value Board_Module -> 70x43
- moved D203 34.3 mm to (-3.00, 5.50), turned to 180 degrees
- moved D202 33.4 mm to (-3.00, 7.00), turned to 180 degrees
- moved R203 32.2 mm to (-5.50, 5.75), turned to 0 degrees
- moved R202 31.3 mm to (-5.50, 6.75), turned to 0 degrees
- moved D200 22.5 mm to (-3.00, -5.50), turned to 180 degrees
- moved R200 19.6 mm to (-5.50, -5.75), turned to 0 degrees
- moved D201 19.2 mm to (-3.00, -7.00), turned to 180 degrees
- moved R201 16.8 mm to (-5.50, -6.75), turned to 0 degrees
- moved J102 13.3 mm to (30.5, -6.00)
- moved J103 10.4 mm to (30.5, 11.0)
- moved C231 8.59 mm to (-13.0, 13.0)
- moved FB201 8.50 mm to (18.0, -13.5)
- moved FB202 8.50 mm to (18.0, -17.0)
- moved FB203 8.50 mm to (18.0, 13.5)
- moved FB204 8.50 mm to (18.0, 17.0)
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Connections:
- net /MA120x0P/CLIP renamed /MA120x0P/nCLIP
- net /MA120x0P/ERROR renamed /MA120x0P/nERROR
- C200 pad 1: +24V -> PVDD
- C201 pad 1: +24V -> PVDD
- C202 pad 1: +24V -> PVDD
- C203 pad 1: +24V -> PVDD
- C204 pad 1: +24V -> PVDD
- C205 pad 1: +24V -> PVDD
- C231 pad 1: +24V -> /VIN
- C232 pad 1: +24V -> PVDD
- D202 pad 1: /MUTE -> /nMUTE
- D203 pad 1: /SHDN -> /MA120x0P/nENABLE
- FB205 pad 1: +24V -> /VIN
- FB205 pad 2: +24V -> PVDD
- J100 pad 1: /I2S_MCLK -> +3V3
- J100 pad 10: Net-(J100-Pad10) -> AVSS
- J100 pad 11: /SPI_MISO -> /I2S_SD1
- J100 pad 12: /SPI_CS -> AVSS
- J100 pad 13: /SPI_SCK -> /I2S_SD0
- J100 pad 14: /SPI_MOSI -> AVSS
- J100 pad 15: /SHDN -> /I2S_LRCLK
- J100 pad 16: /MUTE -> AVSS
- J100 pad 17: AVSS -> /I2S_BCLK
- J100 pad 19: +3V3 -> /I2S_MCLK
- J100 pad 2: AVSS -> +5V
- J100 pad 20: +5V -> AVSS
- J100 pad 3: /I2S_LRCLK -> /nMUTE
- J100 pad 5: /I2S_BCLK -> /ENABLE
- J100 pad 7: /I2S_SDI -> /I2C_SDA
- J100 pad 9: Net-(J100-Pad9) -> /I2C_SCL
- J101 pad 2: +24V -> /VIN
- J102 pad 2: /MA120x0P/OUT0B -> AVSS
- J103 pad 2: /MA120x0P/OUT1A -> AVSS
- R200 pad 1: +5V -> +3V3
- R201 pad 1: +5V -> +3V3
- R202 pad 1: +5V -> +3V3
- R203 pad 1: +5V -> +3V3
- R204 pad 2: /SPI_SCK -> /I2C_SCL
- R205 pad 2: /SPI_MOSI -> /I2C_SDA
- R206 pad 1: +5V -> +3V3
- R208 pad 1: +5V -> +3V3
- U200 pad 21: /I2S_BCLK -> Net-(R218-Pad1)
- U200 pad 22: /I2S_LRCLK -> Net-(R219-Pad1)
- U200 pad 23: /I2S_SDI -> Net-(R217-Pad1)
- U200 pad 32: /I2S_BCLK -> Net-(R220-Pad1)
- U200 pad 33: /SHDN -> /MA120x0P/nENABLE
- U200 pad 34: /MUTE -> /nMUTE
- U200 pad 41: +24V -> PVDD
- U200 pad 42: +24V -> PVDD
- U200 pad 7: +24V -> PVDD
- U200 pad 8: +24V -> PVDD
Routing:
- net /SHDN: track 95.3 -> 0.00 mm, vias 2 -> 0
- net /MUTE: track 92.4 -> 0.00 mm, vias 3 -> 0
- net +3V3: track 0.00 -> 56.1 mm, vias 0 -> 3
- net /SPI_SCK: track 53.9 -> 0.00 mm, vias 2 -> 0
- net /SPI_MOSI: track 53.0 -> 0.00 mm, vias 2 -> 0
- net /I2S_SDI: track 46.3 -> 0.00 mm, vias 2 -> 0
- net /nMUTE: track 0.00 -> 41.6 mm, vias 0 -> 2
- net /MA120x0P/nENABLE: track 0.00 -> 34.3 mm, vias 0 -> 2
- net Net-(R220-Pad1): track 0.00 -> 29.3 mm, vias 0 -> 2
- net /MA120x0P/nERROR: track 30.0 -> 6.90 mm, vias 2 -> 0
- net /I2S_MCLK: track 0.00 -> 22.7 mm
- net /I2C_SDA: track 0.00 -> 21.0 mm
- net /I2C_SCL: track 0.00 -> 21.0 mm
- net /I2S_SD0: track 0.00 -> 20.8 mm
- net /I2S_SD1: track 0.00 -> 20.8 mm
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- added copper zone on F.Cu, net /VIN
- added copper zone on F.Cu, net PVDD
- removed copper zone on F.Cu, net +24V
Other:
- board text added: "EN"
- board text added: "ERR"
- board text removed: "ERROR"
- board text removed: "SHDN"
